Commit message: feat(bringup): unified robot URDF with M65 chassis, D-AIS rail, and RM65 arm (#16)
* feat(bringup): add unified robot URDF with M65 chassis, D-AIS rail, and RM65 arm

- Add omr.urdf.xacro as top-level assembly of all subsystems
- Reorganize URDF into subsystem directories (m65/, dais/, arm/)
- Separate mechanical model (*.model.xacro) from ros2_control config
- Add STL meshes for M65 chassis and D-AIS rail/connector
- Add view_robot.launch.py for unified RViz visualization
- Add ros-humble-joint-state-publisher-gui to Dockerfile
- Update bringup.launch.py to use new ros2_control file paths

* refactor(urdf): rename links for clarity (m65_*, rail_*, arm_*)

- m65: chassis_base_footprint→m65_footprint, chassis_base_link→m65_base, etc.
- dais: dais_base_link→rail_base, dais_slider_link→rail_slider
- arm: base_link→arm_base, Link1~6→arm_link1~6

File: src/omr_bringup/urdf/arm/rm_65.urdf.xacro (robot description, xacro)
@@ -9,5 +9,5 @@
   <!-- <joint name="bottom_joint" type="fixed">
     <origin xyz="0 0 0" rpy="0 0 0" />
-    <parent link="base_link"/>
+    <parent link="arm_base"/>
     <child link="bottom_link"/>
   </joint>
@@ -28,5 +28,5 @@
   </link> -->
   <link
-    name="base_link">
+    name="arm_base">
     <inertial>
       <origin
@@ -49,5 +49,5 @@
       <geometry>
         <mesh
-          filename="package://omr_bringup/urdf/meshes/rm_65_arm/base_link.STL" />
+          filename="package://omr_bringup/urdf/arm/meshes/rm_65_arm/base_link.STL" />
       </geometry>
       <material
@@ -63,10 +63,10 @@
       <geometry>
         <mesh
-          filename="package://omr_bringup/urdf/meshes/rm_65_arm/base_link.STL" />
+          filename="package://omr_bringup/urdf/arm/meshes/rm_65_arm/base_link.STL" />
       </geometry>
     </collision>
   </link>
   <link
-    name="Link1">
+    name="arm_link1">
     <inertial>
       <origin
@@ -89,5 +89,5 @@
       <geometry>
         <mesh
-          filename="package://omr_bringup/urdf/meshes/rm_65_arm/link1.STL" />
+          filename="package://omr_bringup/urdf/arm/meshes/rm_65_arm/link1.STL" />
       </geometry>
       <material
@@ -103,5 +103,5 @@
       <geometry>
         <mesh
-          filename="package://omr_bringup/urdf/meshes/rm_65_arm/link1.STL" />
+          filename="package://omr_bringup/urdf/arm/meshes/rm_65_arm/link1.STL" />
       </geometry>
     </collision>
@@ -114,7 +114,7 @@
       rpy="0 0 0" />
     <parent
-      link="base_link" />
+      link="arm_base" />
     <child
-      link="Link1" />
+      link="arm_link1" />
     <axis
       xyz="0 0 1" />
@@ -126,5 +126,5 @@
   </joint>
   <link
-    name="Link2">
+    name="arm_link2">
     <inertial>
       <origin
@@ -147,5 +147,5 @@
       <geometry>
         <mesh
-          filename="package://omr_bringup/urdf/meshes/rm_65_arm/link2.STL" />
+          filename="package://omr_bringup/urdf/arm/meshes/rm_65_arm/link2.STL" />
       </geometry>
       <material
@@ -161,5 +161,5 @@
       <geometry>
         <mesh
-          filename="package://omr_bringup/urdf/meshes/rm_65_arm/link2.STL" />
+          filename="package://omr_bringup/urdf/arm/meshes/rm_65_arm/link2.STL" />
       </geometry>
     </collision>
@@ -172,7 +172,7 @@
       rpy="1.5708 -1.5708 0" />
     <parent
-      link="Link1" />
+      link="arm_link1" />
     <child
-      link="Link2" />
+      link="arm_link2" />
     <axis
       xyz="0 0 1" />
@@ -184,5 +184,5 @@
   </joint>
   <link
-    name="Link3">
+    name="arm_link3">
     <inertial>
       <origin
@@ -205,5 +205,5 @@
       <geometry>
         <mesh
-          filename="package://omr_bringup/urdf/meshes/rm_65_arm/link3.STL" />
+          filename="package://omr_bringup/urdf/arm/meshes/rm_65_arm/link3.STL" />
       </geometry>
       <material
@@ -219,5 +219,5 @@
       <geometry>
         <mesh
-          filename="package://omr_bringup/urdf/meshes/rm_65_arm/link3.STL" />
+          filename="package://omr_bringup/urdf/arm/meshes/rm_65_arm/link3.STL" />
       </geometry>
     </collision>
@@ -230,7 +230,7 @@
       rpy="0 0 1.5708" />
     <parent
-      link="Link2" />
+      link="arm_link2" />
     <child
-      link="Link3" />
+      link="arm_link3" />
     <axis
       xyz="0 0 1" />
@@ -242,5 +242,5 @@
   </joint>
   <link
-    name="Link4">
+    name="arm_link4">
     <inertial>
       <origin
@@ -263,5 +263,5 @@
       <geometry>
         <mesh
-          filename="package://omr_bringup/urdf/meshes/rm_65_arm/link4.STL" />
+          filename="package://omr_bringup/urdf/arm/meshes/rm_65_arm/link4.STL" />
       </geometry>
       <material
@@ -277,5 +277,5 @@
       <geometry>
         <mesh
-          filename="package://omr_bringup/urdf/meshes/rm_65_arm/link4.STL" />
+          filename="package://omr_bringup/urdf/arm/meshes/rm_65_arm/link4.STL" />
       </geometry>
     </collision>
@@ -288,7 +288,7 @@
       rpy="1.5708 0 0" />
     <parent
-      link="Link3" />
+      link="arm_link3" />
     <child
-      link="Link4" />
+      link="arm_link4" />
     <axis
       xyz="0 0 1" />
@@ -300,5 +300,5 @@
   </joint>
   <link
-    name="Link5">
+    name="arm_link5">
     <inertial>
       <origin
@@ -321,5 +321,5 @@
       <geometry>
         <mesh
-          filename="package://omr_bringup/urdf/meshes/rm_65_arm/link5.STL" />
+          filename="package://omr_bringup/urdf/arm/meshes/rm_65_arm/link5.STL" />
       </geometry>
       <material
@@ -335,5 +335,5 @@
       <geometry>
         <mesh
-          filename="package://omr_bringup/urdf/meshes/rm_65_arm/link5.STL" />
+          filename="package://omr_bringup/urdf/arm/meshes/rm_65_arm/link5.STL" />
       </geometry>
     </collision>
@@ -346,7 +346,7 @@
       rpy="-1.5708 0 0" />
     <parent
-      link="Link4" />
+      link="arm_link4" />
     <child
-      link="Link5" />
+      link="arm_link5" />
     <axis
       xyz="0 0 1" />
@@ -359,5 +359,5 @@
   <xacro:if value="${ link6_type =='Link6' }">
     <link
-      name="Link6">
+      name="arm_link6">
       <inertial>
         <origin
@@ -380,5 +380,5 @@
         <geometry>
           <mesh
-            filename="package://omr_bringup/urdf/meshes/rm_65_arm/link6.STL" />
+            filename="package://omr_bringup/urdf/arm/meshes/rm_65_arm/link6.STL" />
         </geometry>
         <material
@@ -394,5 +394,5 @@
         <geometry>
           <mesh
-            filename="package://omr_bringup/urdf/meshes/rm_65_arm/link6.STL" />
+            filename="package://omr_bringup/urdf/arm/meshes/rm_65_arm/link6.STL" />
         </geometry>
       </collision>
@@ -405,7 +405,7 @@
         rpy="1.5708 0 0" />
       <parent
-        link="Link5" />
+        link="arm_link5" />
       <child
-        link="Link6" />
+        link="arm_link6" />
       <axis
         xyz="0 0 1" />
@@ -419,5 +419,5 @@
   <xacro:if value="${ link6_type =='Link6_6f' }">
     <link
-    name="Link6">
+    name="arm_link6">
     <inertial>
       <origin
@@ -440,5 +440,5 @@
         <geometry>
           <mesh
-            filename="package://omr_bringup/urdf/meshes/rm_65_arm/link6_6f.STL" />
+            filename="package://omr_bringup/urdf/arm/meshes/rm_65_arm/link6_6f.STL" />
         </geometry>
         <material
@@ -454,5 +454,5 @@
         <geometry>
           <mesh
-            filename="package://omr_bringup/urdf/meshes/rm_65_arm/link6_6f.STL" />
+            filename="package://omr_bringup/urdf/arm/meshes/rm_65_arm/link6_6f.STL" />
         </geometry>
       </collision>
@@ -465,7 +465,7 @@
         rpy="1.5708 0 0" />
       <parent
-        link="Link5" />
+        link="arm_link5" />
       <child
-        link="Link6" />
+        link="arm_link6" />
       <axis
         xyz="0 0 1" />
@@ -479,5 +479,5 @@
   <xacro:if value="${ link6_type =='Link6_6fb' }">
     <link
-      name="Link6">
+      name="arm_link6">
       <inertial>
         <origin
@@ -500,5 +500,5 @@
         <geometry>
           <mesh
-            filename="package://omr_bringup/urdf/meshes/rm_65_arm/link6_6fb.STL" />
+            filename="package://omr_bringup/urdf/arm/meshes/rm_65_arm/link6_6fb.STL" />
         </geometry>
         <material
@@ -514,5 +514,5 @@
         <geometry>
           <mesh
-            filename="package://omr_bringup/urdf/meshes/rm_65_arm/link6_6fb.STL" />
+            filename="package://omr_bringup/urdf/arm/meshes/rm_65_arm/link6_6fb.STL" />
         </geometry>
       </collision>
@@ -525,7 +525,7 @@
         rpy="1.5708 0 0" />
       <parent
-        link="Link5" />
+        link="arm_link5" />
       <child
-        link="Link6" />
+        link="arm_link6" />
       <axis
         xyz="0 0 1" />
