Commit message: feat(bringup): add Gazebo Fortress simulation for arm + dais + depth camera
URDF: standalone sim_combined.urdf.xacro with M65+D-AIS+RM65 mechanics,
gz_ros2_control/GazeboSimSystem plugins, gz-sim-sensors-system, depth camera

Launch: simulation.launch.py using gz_sim launch, ros_gz_sim create spawn,
ros_gz_bridge for clock and camera, delayed controller spawners, MoveIt2

Configs: sim_controllers_arm.yaml (100Hz/JTC/position) + dais (50Hz/JTC/velocity)

Dockerfile: ros-humble-ros-gz-sim + ros-humble-gz-ros2-control 0.7.20

Collision: dais.model.xacro rail_base + rail_slider collision tags

File: src/omr_bringup/urdf/dais/dais.model.xacro (robot description, xacro)
@@ -43,4 +43,11 @@
         </material>
       </visual>
+      <collision>
+        <origin xyz="${track_origin_x} ${track_origin_y} ${track_origin_z}"
+                rpy="${track_origin_roll} ${track_origin_pitch} ${track_origin_yaw}"/>
+        <geometry>
+          <mesh filename="${track_mesh}" scale="${mesh_scale} ${mesh_scale} ${mesh_scale}"/>
+        </geometry>
+      </collision>
     </link>
     <!-- dais_slider_link — moving connector plate (STL mesh) -->
@@ -60,4 +67,11 @@
         </material>
       </visual>
+      <collision>
+        <origin xyz="${connector_origin_x} ${connector_origin_y} ${connector_origin_z}"
+                rpy="${connector_origin_roll} ${connector_origin_pitch} ${connector_origin_yaw}"/>
+        <geometry>
+          <mesh filename="${connector_mesh}" scale="${mesh_scale} ${mesh_scale} ${mesh_scale}"/>
+        </geometry>
+      </collision>
     </link>
     <!-- ═══════════════════════════════════════════════════════════ -->
