Commit message: fix(bringup): add SDF-level <gazebo> collision block for m65_footprint

File: src/omr_bringup/urdf/sim_combined.urdf.xacro (robot description, xacro)
@@ -16,4 +16,17 @@
   <xacro:m65_ros2_control_model/>
   <xacro:dais_ros2_control_model/>
+  <!-- ═══════════════════════════════════════════════════════════ -->
+  <!--  Gazebo Fortress: ground collision on root footprint         -->
+  <!--  URDF <collision> is dropped by ros_gz_sim create            -->
+  <!-- ═══════════════════════════════════════════════════════════ -->
+  <gazebo reference="m65_footprint">
+    <collision>
+      <geometry>
+        <box>
+          <size>0.7 0.5 0.35</size>
+        </box>
+      </geometry>
+    </collision>
+  </gazebo>
   <!-- ═══════════════════════════════════════════════════════════ -->
   <!--  Cross-system fixed joints                                   -->
