Commit message: fix(bringup): replace STL collision with box for m65_base (Fortress compat)
Gazebo Fortress ignores STL mesh collisions, causing robot to fall
through ground plane. Replaced with simple box geometry.

File: src/omr_bringup/urdf/m65/m65.model.xacro (robot description, xacro)
@@ -39,8 +39,8 @@
       </visual>
       <collision>
-        <origin xyz="${mesh_origin_x} ${mesh_origin_y} ${mesh_origin_z}"
-                rpy="${mesh_origin_roll} ${mesh_origin_pitch} ${mesh_origin_yaw}"/>
+        <!-- Fortress doesn't handle STL mesh collision well; use box as fallback -->
+        <origin xyz="0 0 -0.15" rpy="0 0 0"/>
         <geometry>
-          <mesh filename="${mesh_file}" scale="${mesh_scale} ${mesh_scale} ${mesh_scale}"/>
+          <box size="0.7 0.5 0.35"/>
         </geometry>
       </collision>

Commit message: fix(bringup): correct m65_base box collision z-origin above ground

File: src/omr_bringup/urdf/m65/m65.model.xacro (robot description, xacro)
@@ -40,5 +40,5 @@
       <collision>
         <!-- Fortress doesn't handle STL mesh collision well; use box as fallback -->
-        <origin xyz="0 0 -0.15" rpy="0 0 0"/>
+        <origin xyz="0 0 0.15" rpy="0 0 0"/>
         <geometry>
           <box size="0.7 0.5 0.35"/>

Commit message: fix(bringup): move box collision from m65_base to m65_footprint
Collision on root link (footprint) is more likely to be recognized
by Gazebo Fortress URDF→SDF conversion than on child links.

File: src/omr_bringup/urdf/m65/m65.model.xacro (robot description, xacro)
@@ -22,4 +22,10 @@
     <!-- ═══════════════════════════════════════════════════════════ -->
     <link name="m65_footprint">
+      <collision>
+        <origin xyz="0 0 0.15" rpy="0 0 0"/>
+        <geometry>
+          <box size="0.7 0.5 0.35"/>
+        </geometry>
+      </collision>
     </link>
     <link name="m65_base">

Commit message: fix(bringup): spawn robot at z=0.3 to verify collision behavior

File: src/omr_bringup/urdf/m65/m65.model.xacro (robot description, xacro)
@@ -44,11 +44,4 @@
         </material>
       </visual>
-      <collision>
-        <!-- Fortress doesn't handle STL mesh collision well; use box as fallback -->
-        <origin xyz="0 0 0.15" rpy="0 0 0"/>
-        <geometry>
-          <box size="0.7 0.5 0.35"/>
-        </geometry>
-      </collision>
     </link>
     <link name="m65_wheel_left">

Commit message: fix(bringup): add mass/inertia to m65_footprint for physics activation

File: src/omr_bringup/urdf/m65/m65.model.xacro (robot description, xacro)
@@ -22,4 +22,8 @@
     <!-- ═══════════════════════════════════════════════════════════ -->
     <link name="m65_footprint">
+      <inertial>
+        <mass value="1.0"/>
+        <inertia ixx="0.1" iyy="0.1" izz="0.1" ixy="0" ixz="0" iyz="0"/>
+      </inertial>
       <collision>
         <origin xyz="0 0 0.15" rpy="0 0 0"/>

Commit message: fix(bringup): full physics simulation with collision, elevation, and CMake install
Root causes fixed:
- empty.sdf has physics type=ignored → created empty_with_physics.sdf
  with dartsim physics and Contact plugin
- URDF <collision> dropped by ros_gz_sim create → used <gazebo>
  collision block with 0.7x0.5x0.9 box + friction surface on root link
- m65_footprint had no mass → added 1kg mass/inertia for physics
- spawn at z=0.075 compensates chassis mesh_origin_z=-0.453 offset
- worlds/ directory not installed → added to CMakeLists.txt

File: src/omr_bringup/urdf/m65/m65.model.xacro (robot description, xacro)
@@ -27,7 +27,7 @@
       </inertial>
       <collision>
-        <origin xyz="0 0 0.15" rpy="0 0 0"/>
+        <origin xyz="0 0 0" rpy="0 0 0"/>
         <geometry>
-          <box size="0.7 0.5 0.35"/>
+          <box size="0.7 0.5 0.9"/>
         </geometry>
       </collision>

File: src/omr_bringup/urdf/sim_combined.urdf.xacro (robot description, xacro)
@@ -19,4 +19,5 @@
   <!--  Gazebo Fortress: ground collision on root footprint         -->
   <!--  URDF <collision> is dropped by ros_gz_sim create            -->
+  <!--  Must use <gazebo> tag which survives URDF→SDF conversion    -->
   <!-- ═══════════════════════════════════════════════════════════ -->
   <gazebo reference="m65_footprint">
@@ -24,7 +25,15 @@
       <geometry>
         <box>
-          <size>0.7 0.5 0.35</size>
+          <size>0.7 0.5 0.9</size>
         </box>
       </geometry>
+      <surface>
+        <friction>
+          <ode>
+            <mu>1.0</mu>
+            <mu2>1.0</mu2>
+          </ode>
+        </friction>
+      </surface>
     </collision>
   </gazebo>

Commit message: fix: Gazebo Fortress simulation — collision, physics, controller merge (#31)
* feat(bringup): add Gazebo Fortress simulation for arm + dais + depth camera

URDF: standalone sim_combined.urdf.xacro with M65+D-AIS+RM65 mechanics,
gz_ros2_control/GazeboSimSystem plugins, gz-sim-sensors-system, depth camera

Launch: simulation.launch.py using gz_sim launch, ros_gz_sim create spawn,
ros_gz_bridge for clock and camera, delayed controller spawners, MoveIt2

Configs: sim_controllers_arm.yaml (100Hz/JTC/position) + dais (50Hz/JTC/velocity)

Dockerfile: ros-humble-ros-gz-sim + ros-humble-gz-ros2-control 0.7.20

Collision: dais.model.xacro rail_base + rail_slider collision tags

* perf(docker): add ros-gz-bridge/sim/ros2-control deps, move LLVM tools to Stage 1 with BuildKit apt cache

- Add ros-humble-ros-gz-bridge, ros-gz-sim, gz-ros2-control to apt install
- Move clangd-19/clang-tidy-19/clang-format-19 from Stage 2 into Stage 1
  so they cache with stable base packages, preventing re-download on
  every base-stage change
- Add BuildKit --mount=type=cache with explicit IDs (apt-cache-dev,
  apt-lib-dev) on both Stage 1 LLVM install and Stage 2 build-essential
- Add wget gnupg to Stage 1 for LLVM key download

* fix(bringup): merge dual gz_ros2_control plugins, add ParameterValue and GZ_SIM_RESOURCE_PATH

- Merge two <gazebo> plugin blocks into one to fix class_loader
  namespace collision (hardware_interface → mock_components)
- Merge sim_controllers_arm.yaml + sim_controllers_dais.yaml into
  sim_controllers_combined.yaml (single controller_manager)
- Wrap robot_description in ParameterValue(value_type=str) to
  prevent YAML parser from misinterpreting XML special chars
- Auto-set GZ_SIM_RESOURCE_PATH via SetEnvironmentVariable for
  Gazebo Fortress package:// → model:// resolution
- Add PythonLaunchDescriptionSource import

* fix(bringup): add dartsim physics world, collision on m65 footprint, spawn elevation

- empty.sdf uses physics type=ignored (no collision/gravity).
  Created empty_with_physics.sdf with type=dartsim and Contact plugin
- Add <gazebo reference="m65_footprint"> collision block with
  0.7×0.5×0.9m box + friction surface (URDF <collision> tag is
  dropped by ros_gz_sim create during URDF→SDF conversion)
- Add mass/inertia to m65_footprint (was empty, Gazebo treated
  model as non-physical without it)
- Spawn at z=0.075m (wheel radius) to compensate for chassis
  mesh_origin_z=-0.453 offset
- Add worlds/ directory to CMakeLists.txt install

File: src/omr_bringup/urdf/m65/m65.model.xacro (robot description, xacro)
@@ -22,4 +22,14 @@
     <!-- ═══════════════════════════════════════════════════════════ -->
     <link name="m65_footprint">
+      <inertial>
+        <mass value="1.0"/>
+        <inertia ixx="0.1" iyy="0.1" izz="0.1" ixy="0" ixz="0" iyz="0"/>
+      </inertial>
+      <collision>
+        <origin xyz="0 0 0" rpy="0 0 0"/>
+        <geometry>
+          <box size="0.7 0.5 0.9"/>
+        </geometry>
+      </collision>
     </link>
     <link name="m65_base">
@@ -38,11 +48,4 @@
         </material>
       </visual>
-      <collision>
-        <origin xyz="${mesh_origin_x} ${mesh_origin_y} ${mesh_origin_z}"
-                rpy="${mesh_origin_roll} ${mesh_origin_pitch} ${mesh_origin_yaw}"/>
-        <geometry>
-          <mesh filename="${mesh_file}" scale="${mesh_scale} ${mesh_scale} ${mesh_scale}"/>
-        </geometry>
-      </collision>
     </link>
     <link name="m65_wheel_left">
